File: Hardware/Can.sch (KiCad schematic (older format))
At the start: 6 parts, among them J5 Conn_01x02_Male, U2 MCP2562-H-SN

Commit message: passive components changed to 0603 and Main connector configuration set
Parts:
- C14, C15: footprint Capacitor_SMD:C_0805_2012Metric -> Capacitor_SMD:C_0603_1608Metric
- R12: footprint Resistor_SMD:R_0805_2012Metric -> Resistor_SMD:R_0603_1608Metric
Changed lines of the file:
@@
 F 0 "C14" H 3842 2146 50  0000 L CNN
 F 1 "100n" H 3842 2055 50  0000 L CNN
-F 2 "Capacitor_SMD:C_0805_2012Metric" H 3750 2100 50  0001 C CNN
+F 2 "Capacitor_SMD:C_0603_1608Metric" H 3750 2100 50  0001 C CNN
 F 3 "~" H 3750 2100 50  0001 C CNN
 	1    3750 2100
@@
 F 0 "R12" H 4309 2996 50  0000 L CNN
 F 1 "R120" H 4309 2905 50  0000 L CNN
-F 2 "Resistor_SMD:R_0805_2012Metric" H 4250 2950 50  0001 C CNN
+F 2 "Resistor_SMD:R_0603_1608Metric" H 4250 2950 50  0001 C CNN
 F 3 "~" H 4250 2950 50  0001 C CNN
 	1    4250 2950
@@
 F 0 "C15" H 2142 3096 50  0000 L CNN
 F 1 "100n" H 2142 3005 50  0000 L CNN
-F 2 "Capacitor_SMD:C_0805_2012Metric" H 2050 3050 50  0001 C CNN
+F 2 "Capacitor_SMD:C_0603_1608Metric" H 2050 3050 50  0001 C CNN
 F 3 "~" H 2050 3050 50  0001 C CNN
 	1    2050 3050
