File: Hardware/Driver.sch (KiCad schematic (older format))
At the start: 16 parts, among them Q44 Q_NMOS_GSD, Q45 Q_NMOS_GSD, Q46 Q_NMOS_GSD, U37 MCP23017_SS

Commit message: passive components changed to 0603 and Main connector configuration set
Parts:
- C35: footprint Capacitor_SMD:C_0805_2012Metric -> Capacitor_SMD:C_0603_1608Metric
- R168, R169, R170, R171, R172, R173, R174, R175, R176, R177, R178: footprint Resistor_SMD:R_0805_2012Metric -> Resistor_SMD:R_0603_1608Metric
Changed lines of the file:
@@
 F 0 "R168" H 1941 1604 50  0000 R CNN
 F 1 "10k" H 1941 1695 50  0000 R CNN
-F 2 "Resistor_SMD:R_0805_2012Metric" H 2000 1650 50  0001 C CNN
+F 2 "Resistor_SMD:R_0603_1608Metric" H 2000 1650 50  0001 C CNN
 F 3 "~" H 2000 1650 50  0001 C CNN
 	1    2000 1650
@@
 F 0 "R169" H 2191 1604 50  0000 R CNN
 F 1 "10k" H 2191 1695 50  0000 R CNN
-F 2 "Resistor_SMD:R_0805_2012Metric" H 2250 1650 50  0001 C CNN
+F 2 "Resistor_SMD:R_0603_1608Metric" H 2250 1650 50  0001 C CNN
 F 3 "~" H 2250 1650 50  0001 C CNN
 	1    2250 1650
@@
 F 0 "C35" H 2842 1396 50  0000 L CNN
 F 1 "C_Small" H 2842 1305 50  0000 L CNN
-F 2 "Capacitor_SMD:C_0805_2012Metric" H 2750 1350 50  0001 C CNN
+F 2 "Capacitor_SMD:C_0603_1608Metric" H 2750 1350 50  0001 C CNN
 F 3 "~" H 2750 1350 50  0001 C CNN
 	1    2750 1350
@@
 F 0 "R170" H 3409 4896 50  0000 L CNN
 F 1 "2k" H 3409 4805 50  0000 L CNN
-F 2 "Resistor_SMD:R_0805_2012Metric" H 3350 4850 50  0001 C CNN
+F 2 "Resistor_SMD:R_0603_1608Metric" H 3350 4850 50  0001 C CNN
 F 3 "~" H 3350 4850 50  0001 C CNN
 	1    3350 4850
@@
 F 0 "R171" H 5159 4896 50  0000 L CNN
 F 1 "2k" H 5159 4805 50  0000 L CNN
-F 2 "Resistor_SMD:R_0805_2012Metric" H 5100 4850 50  0001 C CNN
+F 2 "Resistor_SMD:R_0603_1608Metric" H 5100 4850 50  0001 C CNN
 F 3 "~" H 5100 4850 50  0001 C CNN
 	1    5100 4850
@@
 F 0 "R172" H 6959 4896 50  0000 L CNN
 F 1 "2k" H 6959 4805 50  0000 L CNN
-F 2 "Resistor_SMD:R_0805_2012Metric" H 6900 4850 50  0001 C CNN
+F 2 "Resistor_SMD:R_0603_1608Metric" H 6900 4850 50  0001 C CNN
 F 3 "~" H 6900 4850 50  0001 C CNN
 	1    6900 4850
@@
 F 0 "R173" V 2654 5350 50  0000 C CNN
 F 1 "100R" V 2745 5350 50  0000 C CNN
-F 2 "Resistor_SMD:R_0805_2012Metric" H 2850 5350 50  0001 C CNN
+F 2 "Resistor_SMD:R_0603_1608Metric" H 2850 5350 50  0001 C CNN
 F 3 "~" H 2850 5350 50  0001 C CNN
 	1    2850 5350
@@
 F 0 "R176" H 3059 5546 50  0000 L CNN
 F 1 "10k" H 3059 5455 50  0000 L CNN
-F 2 "Resistor_SMD:R_0805_2012Metric" H 3000 5500 50  0001 C CNN
+F 2 "Resistor_SMD:R_0603_1608Metric" H 3000 5500 50  0001 C CNN
 F 3 "~" H 3000 5500 50  0001 C CNN
 	1    3000 5500
@@
 F 0 "R174" V 4404 5350 50  0000 C CNN
 F 1 "100R" V 4495 5350 50  0000 C CNN
-F 2 "Resistor_SMD:R_0805_2012Metric" H 4600 5350 50  0001 C CNN
+F 2 "Resistor_SMD:R_0603_1608Metric" H 4600 5350 50  0001 C CNN
 F 3 "~" H 4600 5350 50  0001 C CNN
 	1    4600 5350
@@
 F 0 "R177" H 4809 5546 50  0000 L CNN
 F 1 "10k" H 4809 5455 50  0000 L CNN
-F 2 "Resistor_SMD:R_0805_2012Metric" H 4750 5500 50  0001 C CNN
+F 2 "Resistor_SMD:R_0603_1608Metric" H 4750 5500 50  0001 C CNN
 F 3 "~" H 4750 5500 50  0001 C CNN
 	1    4750 5500
@@
 F 0 "R175" V 6204 5350 50  0000 C CNN
 F 1 "100R" V 6295 5350 50  0000 C CNN
-F 2 "Resistor_SMD:R_0805_2012Metric" H 6400 5350 50  0001 C CNN
+F 2 "Resistor_SMD:R_0603_1608Metric" H 6400 5350 50  0001 C CNN
 F 3 "~" H 6400 5350 50  0001 C CNN
 	1    6400 5350
@@
 F 0 "R178" H 6609 5546 50  0000 L CNN
 F 1 "10k" H 6609 5455 50  0000 L CNN
-F 2 "Resistor_SMD:R_0805_2012Metric" H 6550 5500 50  0001 C CNN
+F 2 "Resistor_SMD:R_0603_1608Metric" H 6550 5500 50  0001 C CNN
 F 3 "~" H 6550 5500 50  0001 C CNN
 	1    6550 5500
