File: Hardware/HighCurrent.sch (KiCad schematic (older format))
At the start: 65 parts, among them Q28 Q_PMOS_GSD, Q29 Q_PMOS_GSD, Q30 Q_PMOS_GSD, Q31 Q_PMOS_GSD, Q32 Q_PMOS_GSD, Q33 Q_PMOS_GSD, Q34 Q_NPN_BEC, Q35 Q_NPN_BEC, Q36 Q_NPN_BEC, Q37 Q_NPN_BEC, Q38 Q_NPN_BEC, Q39 Q_NPN_BEC, Q40 Q_PMOS_GSD, Q41 Q_PMOS_GSD, Q42 Q_NPN_BEC, Q43 Q_NPN_BEC, U20 LT6106, U21 LT6106, U22 LT6106, U23 LT6106, U24 LT6106

Commit message: passive components changed to 0603 and Main connector configuration set
Parts:
- R103, R104, R105, R106, R107, R108, R109, R110, R111, R112, R113, R114, R115, R116, R117, R118, R119, R120, R121, R122, R123, R124, R125, R128, R129, R130, R131, R132, R133, R134, R135, R97, R98, R99: footprint Resistor_SMD:R_0805_2012Metric -> Resistor_SMD:R_0603_1608Metric
Changed lines of the file:
@@
 F 0 "R97" V 2696 1350 50  0000 C CNN
 F 1 "100R" V 2605 1350 50  0000 C CNN
-F 2 "Resistor_SMD:R_0805_2012Metric" H 2500 1350 50  0001 C CNN
+F 2 "Resistor_SMD:R_0603_1608Metric" H 2500 1350 50  0001 C CNN
 F 3 "~" H 2500 1350 50  0001 C CNN
 	1    2500 1350
@@
 F 0 "R103" H 3309 1696 50  0000 L CNN
 F 1 "1k" H 3309 1605 50  0000 L CNN
-F 2 "Resistor_SMD:R_0805_2012Metric" H 3250 1650 50  0001 C CNN
+F 2 "Resistor_SMD:R_0603_1608Metric" H 3250 1650 50  0001 C CNN
 F 3 "~" H 3250 1650 50  0001 C CNN
 	1    3250 1650
@@
 F 0 "R98" V 5796 1350 50  0000 C CNN
 F 1 "100R" V 5705 1350 50  0000 C CNN
-F 2 "Resistor_SMD:R_0805_2012Metric" H 5600 1350 50  0001 C CNN
+F 2 "Resistor_SMD:R_0603_1608Metric" H 5600 1350 50  0001 C CNN
 F 3 "~" H 5600 1350 50  0001 C CNN
 	1    5600 1350
@@
 F 0 "R104" H 6409 1696 50  0000 L CNN
 F 1 "1k" H 6409 1605 50  0000 L CNN
-F 2 "Resistor_SMD:R_0805_2012Metric" H 6350 1650 50  0001 C CNN
+F 2 "Resistor_SMD:R_0603_1608Metric" H 6350 1650 50  0001 C CNN
 F 3 "~" H 6350 1650 50  0001 C CNN
 	1    6350 1650
@@
 F 0 "R99" V 8896 1350 50  0000 C CNN
 F 1 "100R" V 8805 1350 50  0000 C CNN
-F 2 "Resistor_SMD:R_0805_2012Metric" H 8700 1350 50  0001 C CNN
+F 2 "Resistor_SMD:R_0603_1608Metric" H 8700 1350 50  0001 C CNN
 F 3 "~" H 8700 1350 50  0001 C CNN
 	1    8700 1350
@@
 F 0 "R105" H 9509 1696 50  0000 L CNN
 F 1 "1k" H 9509 1605 50  0000 L CNN
-F 2 "Resistor_SMD:R_0805_2012Metric" H 9450 1650 50  0001 C CNN
+F 2 "Resistor_SMD:R_0603_1608Metric" H 9450 1650 50  0001 C CNN
 F 3 "~" H 9450 1650 50  0001 C CNN
 	1    9450 1650
@@
 F 0 "R124" V 3046 5550 50  0000 C CNN
 F 1 "100R" V 2955 5550 50  0000 C CNN
-F 2 "Resistor_SMD:R_0805_2012Metric" H 2850 5550 50  0001 C CNN
+F 2 "Resistor_SMD:R_0603_1608Metric" H 2850 5550 50  0001 C CNN
 F 3 "~" H 2850 5550 50  0001 C CNN
 	1    2850 5550
@@
 F 0 "R128" H 3659 5896 50  0000 L CNN
 F 1 "1k" H 3659 5805 50  0000 L CNN
-F 2 "Resistor_SMD:R_0805_2012Metric" H 3600 5850 50  0001 C CNN
+F 2 "Resistor_SMD:R_0603_1608Metric" H 3600 5850 50  0001 C CNN
 F 3 "~" H 3600 5850 50  0001 C CNN
 	1    3600 5850
@@
 F 0 "R130" H 2259 6046 50  0000 L CNN
 F 1 "10k" H 2259 5955 50  0000 L CNN
-F 2 "Resistor_SMD:R_0805_2012Metric" H 2200 6000 50  0001 C CNN
+F 2 "Resistor_SMD:R_0603_1608Metric" H 2200 6000 50  0001 C CNN
 F 3 "~" H 2200 6000 50  0001 C CNN
 	1    2200 6000
@@
 F 0 "R132" V 1454 6400 50  0000 C CNN
 F 1 "1k" V 1545 6400 50  0000 C CNN
-F 2 "Resistor_SMD:R_0805_2012Metric" H 1650 6400 50  0001 C CNN
+F 2 "Resistor_SMD:R_0603_1608Metric" H 1650 6400 50  0001 C CNN
 F 3 "~" H 1650 6400 50  0001 C CNN
 	1    1650 6400
@@
 F 0 "R133" V 4454 6400 50  0000 C CNN
 F 1 "1k" V 4545 6400 50  0000 C CNN
-F 2 "Resistor_SMD:R_0805_2012Metric" H 4650 6400 50  0001 C CNN
+F 2 "Resistor_SMD:R_0603_1608Metric" H 4650 6400 50  0001 C CNN
 F 3 "~" H 4650 6400 50  0001 C CNN
 	1    4650 6400
@@
 F 0 "R131" H 5259 6046 50  0000 L CNN
 F 1 "10k" H 5259 5955 50  0000 L CNN
-F 2 "Resistor_SMD:R_0805_2012Metric" H 5200 6000 50  0001 C CNN
+F 2 "Resistor_SMD:R_0603_1608Metric" H 5200 6000 50  0001 C CNN
 F 3 "~" H 5200 6000 50  0001 C CNN
 	1    5200 6000
@@
 F 0 "R129" H 6659 5896 50  0000 L CNN
 F 1 "1k" H 6659 5805 50  0000 L CNN
-F 2 "Resistor_SMD:R_0805_2012Metric" H 6600 5850 50  0001 C CNN
+F 2 "Resistor_SMD:R_0603_1608Metric" H 6600 5850 50  0001 C CNN
 F 3 "~" H 6600 5850 50  0001 C CNN
 	1    6600 5850
@@
 F 0 "R125" V 6046 5550 50  0000 C CNN
 F 1 "100R" V 5955 5550 50  0000 C CNN
-F 2 "Resistor_SMD:R_0805_2012Metric" H 5850 5550 50  0001 C CNN
+F 2 "Resistor_SMD:R_0603_1608Metric" H 5850 5550 50  0001 C CNN
 F 3 "~" H 5850 5550 50  0001 C CNN
 	1    5850 5550
@@
 F 0 "R107" H 3109 2596 50  0000 L CNN
 F 1 "10k" H 3109 2505 50  0000 L CNN
-F 2 "Resistor_SMD:R_0805_2012Metric" H 3050 2550 50  0001 C CNN
+F 2 "Resistor_SMD:R_0603_1608Metric" H 3050 2550 50  0001 C CNN
 F 3 "~" H 3050 2550 50  0001 C CNN
 	1    3050 2550
@@
 F 0 "R113" V 2304 2950 50  0000 C CNN
 F 1 "1k" V 2395 2950 50  0000 C CNN
-F 2 "Resistor_SMD:R_0805_2012Metric" H 2500 2950 50  0001 C CNN
+F 2 "Resistor_SMD:R_0603_1608Metric" H 2500 2950 50  0001 C CNN
 F 3 "~" H 2500 2950 50  0001 C CNN
 	1    2500 2950
@@
 F 0 "R106" H 1509 2596 50  0000 L CNN
 F 1 "10k" H 1509 2505 50  0000 L CNN
-F 2 "Resistor_SMD:R_0805_2012Metric" H 1450 2550 50  0001 C CNN
+F 2 "Resistor_SMD:R_0603_1608Metric" H 1450 2550 50  0001 C CNN
 F 3 "~" H 1450 2550 50  0001 C CNN
 	1    1450 2550
@@
 F 0 "R112" V 704 2950 50  0000 C CNN
 F 1 "1k" V 795 2950 50  0000 C CNN
-F 2 "Resistor_SMD:R_0805_2012Metric" H 900 2950 50  0001 C CNN
+F 2 "Resistor_SMD:R_0603_1608Metric" H 900 2950 50  0001 C CNN
 F 3 "~" H 900 2950 50  0001 C CNN
 	1    900  2950
@@
 F 0 "R109" H 6209 2596 50  0000 L CNN
 F 1 "10k" H 6209 2505 50  0000 L CNN
-F 2 "Resistor_SMD:R_0805_2012Metric" H 6150 2550 50  0001 C CNN
+F 2 "Resistor_SMD:R_0603_1608Metric" H 6150 2550 50  0001 C CNN
 F 3 "~" H 6150 2550 50  0001 C CNN
 	1    6150 2550
@@
 F 0 "R115" V 5404 2950 50  0000 C CNN
 F 1 "1k" V 5495 2950 50  0000 C CNN
-F 2 "Resistor_SMD:R_0805_2012Metric" H 5600 2950 50  0001 C CNN
+F 2 "Resistor_SMD:R_0603_1608Metric" H 5600 2950 50  0001 C CNN
 F 3 "~" H 5600 2950 50  0001 C CNN
 	1    5600 2950
@@
 F 0 "R108" H 4609 2596 50  0000 L CNN
 F 1 "10k" H 4609 2505 50  0000 L CNN
-F 2 "Resistor_SMD:R_0805_2012Metric" H 4550 2550 50  0001 C CNN
+F 2 "Resistor_SMD:R_0603_1608Metric" H 4550 2550 50  0001 C CNN
 F 3 "~" H 4550 2550 50  0001 C CNN
 	1    4550 2550
@@
 F 0 "R114" V 3804 2950 50  0000 C CNN
 F 1 "1k" V 3895 2950 50  0000 C CNN
-F 2 "Resistor_SMD:R_0805_2012Metric" H 4000 2950 50  0001 C CNN
+F 2 "Resistor_SMD:R_0603_1608Metric" H 4000 2950 50  0001 C CNN
 F 3 "~" H 4000 2950 50  0001 C CNN
 	1    4000 2950
@@
 F 0 "R111" H 9309 2596 50  0000 L CNN
 F 1 "10k" H 9309 2505 50  0000 L CNN
-F 2 "Resistor_SMD:R_0805_2012Metric" H 9250 2550 50  0001 C CNN
+F 2 "Resistor_SMD:R_0603_1608Metric" H 9250 2550 50  0001 C CNN
 F 3 "~" H 9250 2550 50  0001 C CNN
 	1    9250 2550
@@
 F 0 "R117" V 8504 2950 50  0000 C CNN
 F 1 "1k" V 8595 2950 50  0000 C CNN
-F 2 "Resistor_SMD:R_0805_2012Metric" H 8700 2950 50  0001 C CNN
+F 2 "Resistor_SMD:R_0603_1608Metric" H 8700 2950 50  0001 C CNN
 F 3 "~" H 8700 2950 50  0001 C CNN
 	1    8700 2950
@@
 F 0 "R110" H 7709 2596 50  0000 L CNN
 F 1 "10k" H 7709 2505 50  0000 L CNN
-F 2 "Resistor_SMD:R_0805_2012Metric" H 7650 2550 50  0001 C CNN
+F 2 "Resistor_SMD:R_0603_1608Metric" H 7650 2550 50  0001 C CNN
 F 3 "~" H 7650 2550 50  0001 C CNN
 	1    7650 2550
@@
 F 0 "R116" V 6904 2950 50  0000 C CNN
 F 1 "1k" V 6995 2950 50  0000 C CNN
-F 2 "Resistor_SMD:R_0805_2012Metric" H 7100 2950 50  0001 C CNN
+F 2 "Resistor_SMD:R_0603_1608Metric" H 7100 2950 50  0001 C CNN
 F 3 "~" H 7100 2950 50  0001 C CNN
 	1    7100 2950
@@
 F 0 "R118" H 1109 3146 50  0000 L CNN
 F 1 "10k" H 1109 3055 50  0000 L CNN
-F 2 "Resistor_SMD:R_0805_2012Metric" H 1050 3100 50  0001 C CNN
+F 2 "Resistor_SMD:R_0603_1608Metric" H 1050 3100 50  0001 C CNN
 F 3 "~" H 1050 3100 50  0001 C CNN
 	1    1050 3100
@@
 F 0 "R119" H 2709 3146 50  0000 L CNN
 F 1 "10k" H 2709 3055 50  0000 L CNN
-F 2 "Resistor_SMD:R_0805_2012Metric" H 2650 3100 50  0001 C CNN
+F 2 "Resistor_SMD:R_0603_1608Metric" H 2650 3100 50  0001 C CNN
 F 3 "~" H 2650 3100 50  0001 C CNN
 	1    2650 3100
@@
 F 0 "R120" H 4209 3146 50  0000 L CNN
 F 1 "10k" H 4209 3055 50  0000 L CNN
-F 2 "Resistor_SMD:R_0805_2012Metric" H 4150 3100 50  0001 C CNN
+F 2 "Resistor_SMD:R_0603_1608Metric" H 4150 3100 50  0001 C CNN
 F 3 "~" H 4150 3100 50  0001 C CNN
 	1    4150 3100
@@
 F 0 "R121" H 5809 3146 50  0000 L CNN
 F 1 "10k" H 5809 3055 50  0000 L CNN
-F 2 "Resistor_SMD:R_0805_2012Metric" H 5750 3100 50  0001 C CNN
+F 2 "Resistor_SMD:R_0603_1608Metric" H 5750 3100 50  0001 C CNN
 F 3 "~" H 5750 3100 50  0001 C CNN
 	1    5750 3100
@@
 F 0 "R122" H 7309 3146 50  0000 L CNN
 F 1 "10k" H 7309 3055 50  0000 L CNN
-F 2 "Resistor_SMD:R_0805_2012Metric" H 7250 3100 50  0001 C CNN
+F 2 "Resistor_SMD:R_0603_1608Metric" H 7250 3100 50  0001 C CNN
 F 3 "~" H 7250 3100 50  0001 C CNN
 	1    7250 3100
@@
 F 0 "R123" H 8909 3146 50  0000 L CNN
 F 1 "10k" H 8909 3055 50  0000 L CNN
-F 2 "Resistor_SMD:R_0805_2012Metric" H 8850 3100 50  0001 C CNN
+F 2 "Resistor_SMD:R_0603_1608Metric" H 8850 3100 50  0001 C CNN
 F 3 "~" H 8850 3100 50  0001 C CNN
 	1    8850 3100
@@
 F 0 "R135" H 4859 6596 50  0000 L CNN
 F 1 "10k" H 4859 6505 50  0000 L CNN
-F 2 "Resistor_SMD:R_0805_2012Metric" H 4800 6550 50  0001 C CNN
+F 2 "Resistor_SMD:R_0603_1608Metric" H 4800 6550 50  0001 C CNN
 F 3 "~" H 4800 6550 50  0001 C CNN
 	1    4800 6550
@@
 F 0 "R134" H 1859 6596 50  0000 L CNN
 F 1 "10k" H 1859 6505 50  0000 L CNN
-F 2 "Resistor_SMD:R_0805_2012Metric" H 1800 6550 50  0001 C CNN
+F 2 "Resistor_SMD:R_0603_1608Metric" H 1800 6550 50  0001 C CNN
 F 3 "~" H 1800 6550 50  0001 C CNN
 	1    1800 6550
