File: Hardware/IsoINPUT.sch (KiCad schematic (older format))
At the start: 12 parts, among them U29 SFH617A-1, U30 SFH617A-1, U31 SFH617A-1, U32 SFH617A-1

Commit message: passive components changed to 0603 and Main connector configuration set
Parts:
- R152, R153, R154, R155, R156, R157, R158, R159: footprint Resistor_SMD:R_0805_2012Metric -> Resistor_SMD:R_0603_1608Metric
Changed lines of the file:
@@
 F 0 "R152" V 1104 1150 50  0000 C CNN
 F 1 "R_Small" V 1195 1150 50  0000 C CNN
-F 2 "Resistor_SMD:R_0805_2012Metric" H 1300 1150 50  0001 C CNN
+F 2 "Resistor_SMD:R_0603_1608Metric" H 1300 1150 50  0001 C CNN
 F 3 "~" H 1300 1150 50  0001 C CNN
 	1    1300 1150
@@
 F 0 "R154" V 1954 1500 50  0000 C CNN
 F 1 "10k" V 2045 1500 50  0000 C CNN
-F 2 "Resistor_SMD:R_0805_2012Metric" H 2150 1500 50  0001 C CNN
+F 2 "Resistor_SMD:R_0603_1608Metric" H 2150 1500 50  0001 C CNN
 F 3 "~" H 2150 1500 50  0001 C CNN
 	1    2150 1500
@@
 F 0 "R153" V 2654 1150 50  0000 C CNN
 F 1 "R_Small" V 2745 1150 50  0000 C CNN
-F 2 "Resistor_SMD:R_0805_2012Metric" H 2850 1150 50  0001 C CNN
+F 2 "Resistor_SMD:R_0603_1608Metric" H 2850 1150 50  0001 C CNN
 F 3 "~" H 2850 1150 50  0001 C CNN
 	1    2850 1150
@@
 F 0 "R155" V 3504 1500 50  0000 C CNN
 F 1 "10k" V 3595 1500 50  0000 C CNN
-F 2 "Resistor_SMD:R_0805_2012Metric" H 3700 1500 50  0001 C CNN
+F 2 "Resistor_SMD:R_0603_1608Metric" H 3700 1500 50  0001 C CNN
 F 3 "~" H 3700 1500 50  0001 C CNN
 	1    3700 1500
@@
 F 0 "R156" V 1054 2250 50  0000 C CNN
 F 1 "R_Small" V 1145 2250 50  0000 C CNN
-F 2 "Resistor_SMD:R_0805_2012Metric" H 1250 2250 50  0001 C CNN
+F 2 "Resistor_SMD:R_0603_1608Metric" H 1250 2250 50  0001 C CNN
 F 3 "~" H 1250 2250 50  0001 C CNN
 	1    1250 2250
@@
 F 0 "R158" V 1904 2600 50  0000 C CNN
 F 1 "10k" V 1995 2600 50  0000 C CNN
-F 2 "Resistor_SMD:R_0805_2012Metric" H 2100 2600 50  0001 C CNN
+F 2 "Resistor_SMD:R_0603_1608Metric" H 2100 2600 50  0001 C CNN
 F 3 "~" H 2100 2600 50  0001 C CNN
 	1    2100 2600
@@
 F 0 "R157" V 2604 2250 50  0000 C CNN
 F 1 "R_Small" V 2695 2250 50  0000 C CNN
-F 2 "Resistor_SMD:R_0805_2012Metric" H 2800 2250 50  0001 C CNN
+F 2 "Resistor_SMD:R_0603_1608Metric" H 2800 2250 50  0001 C CNN
 F 3 "~" H 2800 2250 50  0001 C CNN
 	1    2800 2250
@@
 F 0 "R159" V 3454 2600 50  0000 C CNN
 F 1 "10k" V 3545 2600 50  0000 C CNN
-F 2 "Resistor_SMD:R_0805_2012Metric" H 3650 2600 50  0001 C CNN
+F 2 "Resistor_SMD:R_0603_1608Metric" H 3650 2600 50  0001 C CNN
 F 3 "~" H 3650 2600 50  0001 C CNN
 	1    3650 2600
