File: Hardware/IsoOUTPUT.sch (KiCad schematic (older format))
At the start: 12 parts, among them U33 SFH617A-1, U34 SFH617A-1, U35 SFH617A-1, U36 SFH617A-1

Commit message: passive components changed to 0603 and Main connector configuration set
Parts:
- R160, R161, R162, R163, R164, R165, R166, R167: footprint Resistor_SMD:R_0805_2012Metric -> Resistor_SMD:R_0603_1608Metric
Changed lines of the file:
@@
 F 0 "R164" H 3659 4096 50  0000 L CNN
 F 1 "10k" H 3659 4005 50  0000 L CNN
-F 2 "Resistor_SMD:R_0805_2012Metric" H 3600 4050 50  0001 C CNN
+F 2 "Resistor_SMD:R_0603_1608Metric" H 3600 4050 50  0001 C CNN
 F 3 "~" H 3600 4050 50  0001 C CNN
 	1    3600 4050
@@
 F 0 "R160" H 3659 3596 50  0000 L CNN
 F 1 "10R" H 3659 3505 50  0000 L CNN
-F 2 "Resistor_SMD:R_0805_2012Metric" H 3600 3550 50  0001 C CNN
+F 2 "Resistor_SMD:R_0603_1608Metric" H 3600 3550 50  0001 C CNN
 F 3 "~" H 3600 3550 50  0001 C CNN
 	1    3600 3550
@@
 F 0 "R165" H 5159 4096 50  0000 L CNN
 F 1 "10k" H 5159 4005 50  0000 L CNN
-F 2 "Resistor_SMD:R_0805_2012Metric" H 5100 4050 50  0001 C CNN
+F 2 "Resistor_SMD:R_0603_1608Metric" H 5100 4050 50  0001 C CNN
 F 3 "~" H 5100 4050 50  0001 C CNN
 	1    5100 4050
@@
 F 0 "R161" H 5159 3596 50  0000 L CNN
 F 1 "10R" H 5159 3505 50  0000 L CNN
-F 2 "Resistor_SMD:R_0805_2012Metric" H 5100 3550 50  0001 C CNN
+F 2 "Resistor_SMD:R_0603_1608Metric" H 5100 3550 50  0001 C CNN
 F 3 "~" H 5100 3550 50  0001 C CNN
 	1    5100 3550
@@
 F 0 "R166" H 6659 4096 50  0000 L CNN
 F 1 "10k" H 6659 4005 50  0000 L CNN
-F 2 "Resistor_SMD:R_0805_2012Metric" H 6600 4050 50  0001 C CNN
+F 2 "Resistor_SMD:R_0603_1608Metric" H 6600 4050 50  0001 C CNN
 F 3 "~" H 6600 4050 50  0001 C CNN
 	1    6600 4050
@@
 F 0 "R162" H 6659 3596 50  0000 L CNN
 F 1 "10R" H 6659 3505 50  0000 L CNN
-F 2 "Resistor_SMD:R_0805_2012Metric" H 6600 3550 50  0001 C CNN
+F 2 "Resistor_SMD:R_0603_1608Metric" H 6600 3550 50  0001 C CNN
 F 3 "~" H 6600 3550 50  0001 C CNN
 	1    6600 3550
@@
 F 0 "R167" H 8159 4096 50  0000 L CNN
 F 1 "10k" H 8159 4005 50  0000 L CNN
-F 2 "Resistor_SMD:R_0805_2012Metric" H 8100 4050 50  0001 C CNN
+F 2 "Resistor_SMD:R_0603_1608Metric" H 8100 4050 50  0001 C CNN
 F 3 "~" H 8100 4050 50  0001 C CNN
 	1    8100 4050
@@
 F 0 "R163" H 8159 3596 50  0000 L CNN
 F 1 "10R" H 8159 3505 50  0000 L CNN
-F 2 "Resistor_SMD:R_0805_2012Metric" H 8100 3550 50  0001 C CNN
+F 2 "Resistor_SMD:R_0603_1608Metric" H 8100 3550 50  0001 C CNN
 F 3 "~" H 8100 3550 50  0001 C CNN
 	1    8100 3550
