File: Hardware/LowCurrent.sch (KiCad schematic (older format))
At the start: 130 parts, among them Q10 Q_NPN_BEC, Q11 Q_NPN_BEC, Q12 Q_PMOS_GSD, Q13 Q_PMOS_GSD, Q14 Q_PMOS_GSD, Q15 Q_PMOS_GSD, Q16 Q_PMOS_GSD, Q17 Q_NPN_BEC, Q18 Q_NPN_BEC, Q19 Q_NPN_BEC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

Commit message: passive components changed to 0603 and Main connector configuration set
Parts:
- R19, R20, R21, R22, R23, R29, R30, R31, R32, R33, R34, R35, R36, R37, R38, R39, R40, R41, R42, R43, R44, R45, R46, R47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: footprint Resistor_SMD:R_0805_2012Metric -> Resistor_SMD:R_0603_1608Metric
