File: Hardware/Multiplexers.sch (KiCad schematic (older format))
At the start: 6 parts, among them U38 74HC4051, U39 74HC4051, U40 74HC4051

Commit message: passive components changed to 0603 and Main connector configuration set
Parts:
- C36, C37, C38: footprint Capacitor_SMD:C_0805_2012Metric -> Capacitor_SMD:C_0603_1608Metric
Changed lines of the file:
@@
 F 0 "C38" H 7392 2996 50  0000 L CNN
 F 1 "100n" H 7392 2905 50  0000 L CNN
-F 2 "Capacitor_SMD:C_0805_2012Metric" H 7300 2950 50  0001 C CNN
+F 2 "Capacitor_SMD:C_0603_1608Metric" H 7300 2950 50  0001 C CNN
 F 3 "~" H 7300 2950 50  0001 C CNN
 	1    7300 2950
@@
 F 0 "C37" H 5542 2996 50  0000 L CNN
 F 1 "100n" H 5542 2905 50  0000 L CNN
-F 2 "Capacitor_SMD:C_0805_2012Metric" H 5450 2950 50  0001 C CNN
+F 2 "Capacitor_SMD:C_0603_1608Metric" H 5450 2950 50  0001 C CNN
 F 3 "~" H 5450 2950 50  0001 C CNN
 	1    5450 2950
@@
 F 0 "C36" H 3742 2996 50  0000 L CNN
 F 1 "100n" H 3742 2905 50  0000 L CNN
-F 2 "Capacitor_SMD:C_0805_2012Metric" H 3650 2950 50  0001 C CNN
+F 2 "Capacitor_SMD:C_0603_1608Metric" H 3650 2950 50  0001 C CNN
 F 3 "~" H 3650 2950 50  0001 C CNN
 	1    3650 2950
