File: Hardware/PDM.kicad_pcb (KiCad board)
At the start: 2 copper layers, 119.4 x 119.4 mm, 354 parts, among them J10 USB_B_Mini, J2 Conn_01x06_Male, J4 Micro_SD_Card_Det_Hirose_DM3AT, J5 Conn_01x02_Male, J6 Conn_01x02_Male, J7 Conn_01x02_Male, J8 Conn_01x02_Male, J9 Conn_01x02_Male, Q1 Q_NMOS_GSD, Q10 Q_NPN_BEC, Q11 Q_NPN_BEC, Q12 Q_PMOS_GSD, Q13 Q_PMOS_GSD, Q14 Q_PMOS_GSD, Q15 Q_PMOS_GSD, Q16 Q_PMOS_GSD, Q17 Q_NPN_BEC, Q18 Q_NPN_BEC, Q19 Q_NPN_BEC, Q2 Q_PMOS_GSD, Q20 Q_NPN_BEC, Q21 Q_NPN_BEC, Q22 Q_PMOS_GSD, Q23 Q_PMOS_GSD, Q24 Q_PMOS_GSD, Q25 Q_NPN_BEC, Q26 Q_NPN_BEC, Q27 Q_NPN_BEC, Q28 Q_PMOS_GSD, Q29 Q_PMOS_GSD, Q3 Q_PMOS_GSD, Q30 Q_PMOS_GSD, Q31 Q_PMOS_GSD, Q32 Q_PMOS_GSD, Q33 Q_PMOS_GSD, Q34 Q_NPN_BEC, Q35 Q_NPN_BEC, Q36 Q_NPN_BEC, Q37 Q_NPN_BEC, Q38 Q_NPN_BEC, Q39 Q_NPN_BEC, Q4 Q_PMOS_GSD, Q40 Q_PMOS_GSD, Q41 Q_PMOS_GSD, Q42 Q_NPN_BEC, Q43 Q_NPN_BEC, Q44 Q_NMOS_GSD, Q45 Q_NMOS_GSD, Q46 Q_NMOS_GSD, Q5 Q_PMOS_GSD, Q6 Q_PMOS_GSD, Q7 Q_NPN_BEC, Q8 Q_NPN_BEC, Q9 Q_NPN_BEC, SW1 SW_Push, U1 STM32F446RETx, U10 LT6106, U11 LT6106, U12 LT6106, U13 LT6106, U14 LT6106, U15 LT6106, U16 LT6106, U17 LT6106, U18 LT6106, U19 LT6106, U2 MCP2562-H-SN, U20 LT6106, U21 LT6106, U22 LT6106, U23 LT6106, U24 LT6106, U25 MCP6001x-LT, U26 MCP6001x-LT, U27 MCP6001x-LT, U28 MCP6001x-LT, U29 SFH617A-1, U3 LM2596S-12, U30 SFH617A-1, U31 SFH617A-1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

Commit message: passive components changed to 0603 and Main connector configuration set
Parts:
- added J1: Conn_01x39_Male, FCI39pin:39pinFCI_ECU, F.Cu at (125.2, 132.4)
- BT1, C20, C24, C26, D2, D3, D4, D5, D6, D7, D8, D9, F1, F2, FB1, L2, L3, U3, U4, U5, U6: moved to B.Cu
- C1, C10, C11, C12, C13, C14, C15, C2, C3, C31, C32, C33, C34, C35, C36, C37, C38, C4, C5, C6, C7, C8, C9: footprint Capacitor_SMD:C_0805_2012Metric -> Capacitor_SMD:C_0603_1608Metric
- C16, C17, C18, C19, C21, C22, C25, C27, C28, C29, C30: footprint Capacitor_SMD:C_0805_2012Metric -> Capacitor_SMD:C_0603_1608Metric; moved to B.Cu
- C23: footprint Capacitor_SMD:CP_Elec_6.3x5.8 -> Capacitor_SMD:C_0603_1608Metric; moved to B.Cu
- R1, R10, R103, R104, R105, R106, R107, R108, R109, R11, R110, R111, R112, R113, R114, R115, R116, R117, R118, R119, R12, R120, R121, R122, R123, R124, R125, R128, R129, R130, R131, R132, R133, R134, R135, R136, R137, R138, R139, R140, R141, R142, R143, R144, R145, R146, R147, R148, R149, R150, R151, R152, R153, R154, R155, R156, R157, R158, R159, R160, R161, R162, R163, R164, R165, R166, R167, R168, R169, R170, R171, R172, R173, R174, R175, R176, R177, R178, R179, R180, R19, R2, R20, R21, R22, R23, R29, R3, R30, R31, R32, R33, R34, R35, R36, R37, R38, R39, R4, R40, R41, R42, R43, R44, R45, R46, R47, R48, R49, R5, R50, R51, R52, R53, R59, R6, R60, R61, R62, R63, R64, R65, R66, R67, R68, R69, R7, R70, R71, R72, R73, R74, R75, R76, R77, R78, R79, R8, R80, R81, R85, R86, R87, R88, R89, R9, R90, R91, R92, R93, R94, R95, R96, R97, R98, R99: footprint Resistor_SMD:R_0805_2012Metric -> Resistor_SMD:R_0603_1608Metric
- R13, R14, R15, R16, R17, R18: footprint Resistor_SMD:R_0805_2012Metric -> Resistor_SMD:R_0603_1608Metric; moved to B.Cu
- moved C28 113.9 mm to (192.5, 81.4)
- moved C27 110.1 mm to (190.6, 81.5)
- moved C16 108.9 mm to (190.0, 130.8), turned to 0 degrees
- moved C17 108.9 mm to (190.0, 132.7), turned to 0 degrees
- moved D2 108.9 mm to (190.0, 142.0)
- moved U5 108.9 mm to (190.0, 75.4), turned to 180 degrees
- moved C18 108.9 mm to (190.0, 128.4), turned to 0 degrees
- moved C19 108.9 mm to (190.0, 126.5), turned to 0 degrees
- moved C26 106.3 mm to (188.7, 87.6), turned to 0 degrees
- moved C24 105.1 mm to (188.1, 120.7), turned to 0 degrees
- moved D3 105.1 mm to (188.1, 135.9), turned to 0 degrees
- moved L3 102.3 mm to (186.7, 97.8), turned to 180 degrees
- moved FB1 101.2 mm to (186.2, 129.7)
- moved D9 100.8 mm to (185.9, 81.8), turned to 180 degrees
- moved F1 100.0 mm to (185.5, 142.0)
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Connections:
- net SWGND renamed GND
Routing:
- added copper zone on F.Cu, net VDD
