File: Hardware/Temp_sense.sch (KiCad schematic (older format))
At the start: 32 parts, among them J6 Conn_01x02_Male, J7 Conn_01x02_Male, J8 Conn_01x02_Male, J9 Conn_01x02_Male, U25 MCP6001x-LT, U26 MCP6001x-LT, U27 MCP6001x-LT, U28 MCP6001x-LT

Commit message: passive components changed to 0603 and Main connector configuration set
Parts:
- C31, C32, C33, C34: footprint Capacitor_SMD:C_0805_2012Metric -> Capacitor_SMD:C_0603_1608Metric
- R136, R137, R138, R139, R140, R141, R142, R143, R144, R145, R146, R147, R148, R149, R150, R151: footprint Resistor_SMD:R_0805_2012Metric -> Resistor_SMD:R_0603_1608Metric
Changed lines of the file:
@@
 F 0 "R140" H 1709 2446 50  0000 L CNN
 F 1 "10k" H 1709 2355 50  0000 L CNN
-F 2 "Resistor_SMD:R_0805_2012Metric" H 1650 2400 50  0001 C CNN
+F 2 "Resistor_SMD:R_0603_1608Metric" H 1650 2400 50  0001 C CNN
 F 3 "~" H 1650 2400 50  0001 C CNN
 	1    1650 2400
@@
 F 0 "R142" H 2659 2696 50  0000 L CNN
 F 1 "10k" H 2659 2605 50  0000 L CNN
-F 2 "Resistor_SMD:R_0805_2012Metric" H 2600 2650 50  0001 C CNN
+F 2 "Resistor_SMD:R_0603_1608Metric" H 2600 2650 50  0001 C CNN
 F 3 "~" H 2600 2650 50  0001 C CNN
 	1    2600 2650
@@
 F 0 "C31" H 3742 2196 50  0000 L CNN
 F 1 "100nF" H 3742 2105 50  0000 L CNN
-F 2 "Capacitor_SMD:C_0805_2012Metric" H 3650 2150 50  0001 C CNN
+F 2 "Capacitor_SMD:C_0603_1608Metric" H 3650 2150 50  0001 C CNN
 F 3 "~" H 3650 2150 50  0001 C CNN
 	1    3650 2150
@@
 F 0 "R138" H 3559 2046 50  0000 L CNN
 F 1 "10k" H 3559 1955 50  0000 L CNN
-F 2 "Resistor_SMD:R_0805_2012Metric" H 3500 2000 50  0001 C CNN
+F 2 "Resistor_SMD:R_0603_1608Metric" H 3500 2000 50  0001 C CNN
 F 3 "~" H 3500 2000 50  0001 C CNN
 	1    3500 2000
@@
 F 0 "R141" H 5259 2446 50  0000 L CNN
 F 1 "10k" H 5259 2355 50  0000 L CNN
-F 2 "Resistor_SMD:R_0805_2012Metric" H 5200 2400 50  0001 C CNN
+F 2 "Resistor_SMD:R_0603_1608Metric" H 5200 2400 50  0001 C CNN
 F 3 "~" H 5200 2400 50  0001 C CNN
 	1    5200 2400
@@
 F 0 "R143" H 6209 2696 50  0000 L CNN
 F 1 "10k" H 6209 2605 50  0000 L CNN
-F 2 "Resistor_SMD:R_0805_2012Metric" H 6150 2650 50  0001 C CNN
+F 2 "Resistor_SMD:R_0603_1608Metric" H 6150 2650 50  0001 C CNN
 F 3 "~" H 6150 2650 50  0001 C CNN
 	1    6150 2650
@@
 F 0 "R139" H 7109 2046 50  0000 L CNN
 F 1 "10k" H 7109 1955 50  0000 L CNN
-F 2 "Resistor_SMD:R_0805_2012Metric" H 7050 2000 50  0001 C CNN
+F 2 "Resistor_SMD:R_0603_1608Metric" H 7050 2000 50  0001 C CNN
 F 3 "~" H 7050 2000 50  0001 C CNN
 	1    7050 2000
@@
 F 0 "R149" H 1709 4146 50  0000 L CNN
 F 1 "10k" H 1709 4055 50  0000 L CNN
-F 2 "Resistor_SMD:R_0805_2012Metric" H 1650 4100 50  0001 C CNN
+F 2 "Resistor_SMD:R_0603_1608Metric" H 1650 4100 50  0001 C CNN
 F 3 "~" H 1650 4100 50  0001 C CNN
 	1    1650 4100
@@
 F 0 "R151" H 2659 4396 50  0000 L CNN
 F 1 "10k" H 2659 4305 50  0000 L CNN
-F 2 "Resistor_SMD:R_0805_2012Metric" H 2600 4350 50  0001 C CNN
+F 2 "Resistor_SMD:R_0603_1608Metric" H 2600 4350 50  0001 C CNN
 F 3 "~" H 2600 4350 50  0001 C CNN
 	1    2600 4350
@@
 F 0 "R147" H 3559 3746 50  0000 L CNN
 F 1 "10k" H 3559 3655 50  0000 L CNN
-F 2 "Resistor_SMD:R_0805_2012Metric" H 3500 3700 50  0001 C CNN
+F 2 "Resistor_SMD:R_0603_1608Metric" H 3500 3700 50  0001 C CNN
 F 3 "~" H 3500 3700 50  0001 C CNN
 	1    3500 3700
@@
 F 0 "R148" H 5259 4096 50  0000 L CNN
 F 1 "10k" H 5259 4005 50  0000 L CNN
-F 2 "Resistor_SMD:R_0805_2012Metric" H 5200 4050 50  0001 C CNN
+F 2 "Resistor_SMD:R_0603_1608Metric" H 5200 4050 50  0001 C CNN
 F 3 "~" H 5200 4050 50  0001 C CNN
 	1    5200 4050
@@
 F 0 "R150" H 6209 4346 50  0000 L CNN
 F 1 "10k" H 6209 4255 50  0000 L CNN
-F 2 "Resistor_SMD:R_0805_2012Metric" H 6150 4300 50  0001 C CNN
+F 2 "Resistor_SMD:R_0603_1608Metric" H 6150 4300 50  0001 C CNN
 F 3 "~" H 6150 4300 50  0001 C CNN
 	1    6150 4300
@@
 F 0 "R146" H 7109 3696 50  0000 L CNN
 F 1 "10k" H 7109 3605 50  0000 L CNN
-F 2 "Resistor_SMD:R_0805_2012Metric" H 7050 3650 50  0001 C CNN
+F 2 "Resistor_SMD:R_0603_1608Metric" H 7050 3650 50  0001 C CNN
 F 3 "~" H 7050 3650 50  0001 C CNN
 	1    7050 3650
@@
 F 0 "R136" H 1409 1946 50  0000 L CNN
 F 1 "10R" H 1409 1855 50  0000 L CNN
-F 2 "Resistor_SMD:R_0805_2012Metric" H 1350 1900 50  0001 C CNN
+F 2 "Resistor_SMD:R_0603_1608Metric" H 1350 1900 50  0001 C CNN
 F 3 "~" H 1350 1900 50  0001 C CNN
 	1    1350 1900
@@
 F 0 "R137" H 4959 1946 50  0000 L CNN
 F 1 "10R" H 4959 1855 50  0000 L CNN
-F 2 "Resistor_SMD:R_0805_2012Metric" H 4900 1900 50  0001 C CNN
+F 2 "Resistor_SMD:R_0603_1608Metric" H 4900 1900 50  0001 C CNN
 F 3 "~" H 4900 1900 50  0001 C CNN
 	1    4900 1900
@@
 F 0 "R145" H 1409 3646 50  0000 L CNN
 F 1 "10R" H 1409 3555 50  0000 L CNN
-F 2 "Resistor_SMD:R_0805_2012Metric" H 1350 3600 50  0001 C CNN
+F 2 "Resistor_SMD:R_0603_1608Metric" H 1350 3600 50  0001 C CNN
 F 3 "~" H 1350 3600 50  0001 C CNN
 	1    1350 3600
@@
 F 0 "R144" H 4959 3596 50  0000 L CNN
 F 1 "10R" H 4959 3505 50  0000 L CNN
-F 2 "Resistor_SMD:R_0805_2012Metric" H 4900 3550 50  0001 C CNN
+F 2 "Resistor_SMD:R_0603_1608Metric" H 4900 3550 50  0001 C CNN
 F 3 "~" H 4900 3550 50  0001 C CNN
 	1    4900 3550
@@
 F 0 "C32" H 7292 2196 50  0000 L CNN
 F 1 "100nF" H 7292 2105 50  0000 L CNN
-F 2 "Capacitor_SMD:C_0805_2012Metric" H 7200 2150 50  0001 C CNN
+F 2 "Capacitor_SMD:C_0603_1608Metric" H 7200 2150 50  0001 C CNN
 F 3 "~" H 7200 2150 50  0001 C CNN
 	1    7200 2150
@@
 F 0 "C33" H 7292 3846 50  0000 L CNN
 F 1 "100nF" H 7292 3755 50  0000 L CNN
-F 2 "Capacitor_SMD:C_0805_2012Metric" H 7200 3800 50  0001 C CNN
+F 2 "Capacitor_SMD:C_0603_1608Metric" H 7200 3800 50  0001 C CNN
 F 3 "~" H 7200 3800 50  0001 C CNN
 	1    7200 3800
@@
 F 0 "C34" H 3742 3896 50  0000 L CNN
 F 1 "100nF" H 3742 3805 50  0000 L CNN
-F 2 "Capacitor_SMD:C_0805_2012Metric" H 3650 3850 50  0001 C CNN
+F 2 "Capacitor_SMD:C_0603_1608Metric" H 3650 3850 50  0001 C CNN
 F 3 "~" H 3650 3850 50  0001 C CNN
 	1    3650 3850
