File: Hardware/USB.sch (KiCad schematic (older format))
At the start: 3 parts, among them J10 USB_B_Mini

Commit message: passive components changed to 0603 and Main connector configuration set
Parts:
- R179, R180: footprint Resistor_SMD:R_0805_2012Metric -> Resistor_SMD:R_0603_1608Metric
Changed lines of the file:
@@
 F 0 "R179" V 2954 2850 50  0000 C CNN
 F 1 "10R" V 3045 2850 50  0000 C CNN
-F 2 "Resistor_SMD:R_0805_2012Metric" H 3150 2850 50  0001 C CNN
+F 2 "Resistor_SMD:R_0603_1608Metric" H 3150 2850 50  0001 C CNN
 F 3 "~" H 3150 2850 50  0001 C CNN
 	1    3150 2850
@@
 F 0 "R180" V 2954 2950 50  0000 C CNN
 F 1 "10R" V 3045 2950 50  0000 C CNN
-F 2 "Resistor_SMD:R_0805_2012Metric" H 3150 2950 50  0001 C CNN
+F 2 "Resistor_SMD:R_0603_1608Metric" H 3150 2950 50  0001 C CNN
 F 3 "~" H 3150 2950 50  0001 C CNN
 	1    3150 2950
