File: Hardware/sdCard.sch (KiCad schematic (older format))
At the start: 8 parts, among them J4 Micro_SD_Card_Det_Hirose_DM3AT

Commit message: passive components changed to 0603 and Main connector configuration set
Parts:
- C13: footprint Capacitor_SMD:C_0805_2012Metric -> Capacitor_SMD:C_0603_1608Metric
- R10, R11, R6, R7, R8, R9: footprint Resistor_SMD:R_0805_2012Metric -> Resistor_SMD:R_0603_1608Metric
Changed lines of the file:
@@
 F 0 "R6" H 3259 2846 50  0000 L CNN
 F 1 "47k" H 3259 2755 50  0000 L CNN
-F 2 "Resistor_SMD:R_0805_2012Metric" H 3200 2800 50  0001 C CNN
+F 2 "Resistor_SMD:R_0603_1608Metric" H 3200 2800 50  0001 C CNN
 F 3 "~" H 3200 2800 50  0001 C CNN
 	1    3200 2800
@@
 F 0 "R7" H 3559 2846 50  0000 L CNN
 F 1 "47k" H 3559 2755 50  0000 L CNN
-F 2 "Resistor_SMD:R_0805_2012Metric" H 3500 2800 50  0001 C CNN
+F 2 "Resistor_SMD:R_0603_1608Metric" H 3500 2800 50  0001 C CNN
 F 3 "~" H 3500 2800 50  0001 C CNN
 	1    3500 2800
@@
 F 0 "R8" H 3859 2846 50  0000 L CNN
 F 1 "47k" H 3859 2755 50  0000 L CNN
-F 2 "Resistor_SMD:R_0805_2012Metric" H 3800 2800 50  0001 C CNN
+F 2 "Resistor_SMD:R_0603_1608Metric" H 3800 2800 50  0001 C CNN
 F 3 "~" H 3800 2800 50  0001 C CNN
 	1    3800 2800
@@
 F 0 "R9" H 4359 2846 50  0000 L CNN
 F 1 "47k" H 4359 2755 50  0000 L CNN
-F 2 "Resistor_SMD:R_0805_2012Metric" H 4300 2800 50  0001 C CNN
+F 2 "Resistor_SMD:R_0603_1608Metric" H 4300 2800 50  0001 C CNN
 F 3 "~" H 4300 2800 50  0001 C CNN
 	1    4300 2800
@@
 F 0 "R10" H 4859 2846 50  0000 L CNN
 F 1 "47k" H 4859 2755 50  0000 L CNN
-F 2 "Resistor_SMD:R_0805_2012Metric" H 4800 2800 50  0001 C CNN
+F 2 "Resistor_SMD:R_0603_1608Metric" H 4800 2800 50  0001 C CNN
 F 3 "~" H 4800 2800 50  0001 C CNN
 	1    4800 2800
@@
 F 0 "R11" H 4609 3996 50  0000 L CNN
 F 1 "180k" H 4609 3905 50  0000 L CNN
-F 2 "Resistor_SMD:R_0805_2012Metric" H 4550 3950 50  0001 C CNN
+F 2 "Resistor_SMD:R_0603_1608Metric" H 4550 3950 50  0001 C CNN
 F 3 "~" H 4550 3950 50  0001 C CNN
 	1    4550 3950
@@
 F 0 "C13" H 4158 2304 50  0000 R CNN
 F 1 "100nF" H 4158 2395 50  0000 R CNN
-F 2 "Capacitor_SMD:C_0805_2012Metric" H 4250 2350 50  0001 C CNN
+F 2 "Capacitor_SMD:C_0603_1608Metric" H 4250 2350 50  0001 C CNN
 F 3 "~" H 4250 2350 50  0001 C CNN
 	1    4250 2350
